File: beacon.sch (KiCad schematic (older format))
At the start: 64 parts, among them SW1 RST, U1 NUF2042XV6, U2 SN65HVD256, U3 MPU-9250, U4 LT1965-3.3, U5 STM32F405RGT6, U6 DWM1000, X1 16MHz

Commit message: Make it possible to boot from DFU
Fixes #1
Parts:
- added R11, R12: 10k, symbol device1:R_Small
- added SW2: DFU, symbol _div:PushButton_B3U
- C1, C10, C11, C12, C13, C14, C15, C16, C17, C18, C2, C3, C4, C5, C6, C7, C8, C9: symbol C_Small -> device1:C_Small
- CONN1: symbol MICRO_USB -> _connectors:MICRO_USB
- CONN2, CONN3: symbol CAN -> _connectors:CAN
- CONN4: symbol SWD/DEBUG -> beacon-rescue:SWD_DEBUG-RESCUE-beacon
- D1, D2: symbol D_Schottky_Small -> device1:D_Schottky_Small
- D10, D3, D4, D5, D6, D7, D8, D9: symbol Led_Small -> beacon-rescue:Led_Small-RESCUE-beacon
- F1, F2: symbol F_Small -> beacon-rescue:F_Small-RESCUE-beacon
- H1, H2, H3, H4: symbol HOLE -> cvra:HOLE
- R1, R10, R2, R3, R4, R5, R6, R7, R8, R9: symbol R_Small -> device1:R_Small
- SW1: symbol SW_PUSH_SMALL -> beacon-rescue:SW_PUSH_SMALL-RESCUE-beacon
- U1: symbol NUF2042XV6 -> _div:NUF2042XV6
- U2: symbol SN65HVD256 -> _transceiver:SN65HVD256
- U3: symbol MPU-9250 -> _sensors:MPU-9250
- U4: symbol LT1965 -> _linear-regulators:LT1965
- U5: symbol STM32F415RGT6 -> _stm32:STM32F415RGT6
- U6: symbol DWM1000 -> _wireless:DWM1000
- W1, W2, W3, W4, W5, W6, W7, W8: symbol TEST_1P -> beacon-rescue:TEST_1P-RESCUE-beacon
- X1: symbol XTAL-SMD-4-PADS -> _div:XTAL-SMD-4-PADS
Connections:
- net labels added: BOOT0, BOOT1
- wire segments 225 -> 296
- no-connect marks 45 -> 44
Other:
- note added: "Boot config:\n- Button pushed: DFU bootloader\n- Button released: boot from flash"
- note removed: "Boot from \nflash"

Commit message: Move status LED pins
Parts:
- R11, R12: footprint (none) -> _std:R_0603
- SW2: footprint (none) -> _div:SMD_Pushbutton_B3U-3100P
Changed lines of the file:
@@
 NoConn ~ 3525 1525
 NoConn ~ 3525 2325
-NoConn ~ 3525 2925
 NoConn ~ 3525 3525
 NoConn ~ 3525 3625
@@
 NoConn ~ 3525 5125
 NoConn ~ 3525 5225
-NoConn ~ 3525 5325
 NoConn ~ 3525 5425
 NoConn ~ 3525 5525
@@
 NoConn ~ 3525 6325
 NoConn ~ 3525 6525
+Text Label 3950 5325 2    39   ~ 0
+ERROR_LED
 Text Label 3950 3125 2    39   ~ 0
-ERROR_LED
+DEBUG_LED
 Text Label 3950 3225 2    39   ~ 0
-DEBUG_LED
-Text Label 3950 3425 2    39   ~ 0
 STATUS_LED
 $Comp
@@
 Connection ~ 2000 1925
 Wire Wire Line
+	3950 5325 3525 5325
+Wire Wire Line
 	3950 3125 3525 3125
-Wire Wire Line
-	3950 3225 3525 3225
 Wire Wire Line
 	10625 4725 10625 4875
@@
 L beacon-rescue:TEST_1P-RESCUE-beacon W1
 U 1 1 57728662
-P 4375 5225
-F 0 "W1" H 4375 5275 31  0000 L CNN
-F 1 "TEST_UWB_CSN" H 4425 5350 31  0000 L CNN
-F 2 "_div:Test_1pin_SMD" H 4575 5225 50  0001 C CNN
-F 3 "" H 4575 5225 50  0000 C CNN
-	1    4375 5225
-	1    0    0    -1
-$EndComp
-Text Label 3950 5225 0    39   ~ 0
+P 4625 5375
+F 0 "W1" H 4625 5425 31  0000 L CNN
+F 1 "TEST_UWB_CSN" H 4675 5500 31  0000 L CNN
+F 2 "_div:Test_1pin_SMD" H 4825 5375 50  0001 C CNN
+F 3 "" H 4825 5375 50  0000 C CNN
+	1    4625 5375
+	1    0    0    -1
+$EndComp
+Text Label 4200 5375 0    39   ~ 0
 UWB_CS_N
-Text Label 3950 5525 0    39   ~ 0
+Text Label 4200 5675 0    39   ~ 0
 UWB_MOSI
-Text Label 3950 5425 0    39   ~ 0
+Text Label 4200 5575 0    39   ~ 0
 UWB_MISO
-Text Label 3950 5325 0    39   ~ 0
+Text Label 4200 5475 0    39   ~ 0
 UWB_CLK
 Wire Wire Line
-	3950 5225 4375 5225
-Wire Wire Line
-	3950 5525 4750 5525
-Wire Wire Line
-	3950 5425 4625 5425
-Wire Wire Line
-	3950 5325 4500 5325
+	4200 5375 4625 5375
+Wire Wire Line
+	4200 5675 5000 5675
+Wire Wire Line
+	4200 5575 4875 5575
 $Comp
 L beacon-rescue:TEST_1P-RESCUE-beacon W2
 U 1 1 5772BF67
-P 4500 5325
-F 0 "W2" H 4500 5375 31  0000 L CNN
-F 1 "TEST_UWB_CLK" H 4550 5450 31  0000 L CNN
-F 2 "_div:Test_1pin_SMD" H 4700 5325 50  0001 C CNN
-F 3 "" H 4700 5325 50  0000 C CNN
-	1    4500 5325
+P 4750 5475
+F 0 "W2" H 4750 5525 31  0000 L CNN
+F 1 "TEST_UWB_CLK" H 4800 5600 31  0000 L CNN
+F 2 "_div:Test_1pin_SMD" H 4950 5475 50  0001 C CNN
+F 3 "" H 4950 5475 50  0000 C CNN
+	1    4750 5475
 	1    0    0    -1
 $EndComp
@@
 L beacon-rescue:TEST_1P-RESCUE-beacon W3
 U 1 1 5772C1F8
-P 4625 5425
-F 0 "W3" H 4625 5475 31  0000 L CNN
-F 1 "TEST_UWB_MISO" H 4675 5550 31  0000 L CNN
-F 2 "_div:Test_1pin_SMD" H 4825 5425 50  0001 C CNN
-F 3 "" H 4825 5425 50  0000 C CNN
-	1    4625 5425
+P 4875 5575
+F 0 "W3" H 4875 5625 31  0000 L CNN
+F 1 "TEST_UWB_MISO" H 4925 5700 31  0000 L CNN
+F 2 "_div:Test_1pin_SMD" H 5075 5575 50  0001 C CNN
+F 3 "" H 5075 5575 50  0000 C CNN
+	1    4875 5575
 	1    0    0    -1
 $EndComp
@@
 L beacon-rescue:TEST_1P-RESCUE-beacon W4
 U 1 1 5772C2C5
-P 4750 5525
-F 0 "W4" H 4750 5575 31  0000 L CNN
-F 1 "TEST_UWB_MOSI" H 4800 5650 31  0000 L CNN
-F 2 "_div:Test_1pin_SMD" H 4950 5525 50  0001 C CNN
-F 3 "" H 4950 5525 50  0000 C CNN
-	1    4750 5525
-	1    0    0    -1
-$EndComp
-Text Label 3950 5875 0    39   ~ 0
+P 5000 5675
+F 0 "W4" H 5000 5725 31  0000 L CNN
+F 1 "TEST_UWB_MOSI" H 5050 5800 31  0000 L CNN
+F 2 "_div:Test_1pin_SMD" H 5200 5675 50  0001 C CNN
+F 3 "" H 5200 5675 50  0000 C CNN
+	1    5000 5675
+	1    0    0    -1
+$EndComp
+Text Label 4200 6025 0    39   ~ 0
 IMU_SCK
-Text Label 3950 6075 0    39   ~ 0
+Text Label 4200 6225 0    39   ~ 0
 IMU_MOSI
-Text Label 3950 5975 0    39   ~ 0
+Text Label 4200 6125 0    39   ~ 0
 IMU_MISO
-Text Label 3950 5775 0    39   ~ 0
+Text Label 4200 5925 0    39   ~ 0
 IMU_CS_N
 Wire Wire Line
-	3950 5875 4500 5875
-Wire Wire Line
-	3950 6075 4750 6075
-Wire Wire Line
-	3950 5975 4625 5975
-Wire Wire Line
-	3950 5775 4375 5775
+	4200 6025 4750 6025
+Wire Wire Line
+	4200 6225 5000 6225
+Wire Wire Line
+	4200 6125 4875 6125
+Wire Wire Line
+	4200 5925 4625 5925
 $Comp
 L beacon-rescue:TEST_1P-RESCUE-beacon W5
 U 1 1 5772D51D
-P 4375 5775
-F 0 "W5" H 4375 5825 31  0000 L CNN
-F 1 "TEST_IMU_CSN" H 4425 5900 31  0000 L CNN
-F 2 "_div:Test_1pin_SMD" H 4575 5775 50  0001 C CNN
-F 3 "" H 4575 5775 50  0000 C CNN
-	1    4375 5775
+P 4625 5925
+F 0 "W5" H 4625 5975 31  0000 L CNN
+F 1 "TEST_IMU_CSN" H 4675 6050 31  0000 L CNN
+F 2 "_div:Test_1pin_SMD" H 4825 5925 50  0001 C CNN
+F 3 "" H 4825 5925 50  0000 C CNN
+	1    4625 5925
 	1    0    0    -1
 $EndComp
@@
 L beacon-rescue:TEST_1P-RESCUE-beacon W6
 U 1 1 5772D68C
-P 4500 5875
-F 0 "W6" H 4500 5925 31  0000 L CNN
-F 1 "TEST_UWB_SCK" H 4550 6000 31  0000 L CNN
-F 2 "_div:Test_1pin_SMD" H 4700 5875 50  0001 C CNN
-F 3 "" H 4700 5875 50  0000 C CNN
-	1    4500 5875
+P 4750 6025
+F 0 "W6" H 4750 6075 31  0000 L CNN
+F 1 "TEST_UWB_SCK" H 4800 6150 31  0000 L CNN
+F 2 "_div:Test_1pin_SMD" H 4950 6025 50  0001 C CNN
+F 3 "" H 4950 6025 50  0000 C CNN
+	1    4750 6025
 	1    0    0    -1
 $EndComp
@@
 L beacon-rescue:TEST_1P-RESCUE-beacon W7
 U 1 1 5772DE24
-P 4625 5975
-F 0 "W7" H 4625 6025 31  0000 L CNN
-F 1 "TEST_UWB_MISO" H 4675 6100 31  0000 L CNN
-F 2 "_div:Test_1pin_SMD" H 4825 5975 50  0001 C CNN
-F 3 "" H 4825 5975 50  0000 C CNN
-	1    4625 5975
+P 4875 6125
+F 0 "W7" H 4875 6175 31  0000 L CNN
+F 1 "TEST_UWB_MISO" H 4925 6250 31  0000 L CNN
+F 2 "_div:Test_1pin_SMD" H 5075 6125 50  0001 C CNN
+F 3 "" H 5075 6125 50  0000 C CNN
+	1    4875 6125
 	1    0    0    -1
 $EndComp
@@
 L beacon-rescue:TEST_1P-RESCUE-beacon W8
 U 1 1 5772DEF1
-P 4750 6075
-F 0 "W8" H 4750 6125 31  0000 L CNN
-F 1 "TEST_UWB_MOSI" H 4800 6200 31  0000 L CNN
-F 2 "_div:Test_1pin_SMD" H 4950 6075 50  0001 C CNN
-F 3 "" H 4950 6075 50  0000 C CNN
-	1    4750 6075
+P 5000 6225
+F 0 "W8" H 5000 6275 31  0000 L CNN
+F 1 "TEST_UWB_MOSI" H 5050 6350 31  0000 L CNN
+F 2 "_div:Test_1pin_SMD" H 5200 6225 50  0001 C CNN
+F 3 "" H 5200 6225 50  0000 C CNN
+	1    5000 6225
 	1    0    0    -1
 $EndComp
@@
 BOOT1
 Wire Wire Line
-	3950 3425 3525 3425
-Wire Wire Line
 	3950 3325 3525 3325
 Text Label 1825 1525 0    39   ~ 0
@@
 F 0 "R12" V 1500 4975 39  0000 C CNN
 F 1 "10k" V 1425 4975 39  0000 C CNN
-F 2 "" H 1425 4975 50  0001 C CNN
+F 2 "_std:R_0603" H 1425 4975 50  0001 C CNN
 F 3 "" H 1425 4975 50  0001 C CNN
 	1    1425 4975
@@
 F 0 "R11" V 1500 4825 39  0000 C CNN
 F 1 "10k" V 1425 4825 39  0000 C CNN
-F 2 "" H 1425 4825 50  0001 C CNN
+F 2 "_std:R_0603" H 1425 4825 50  0001 C CNN
 F 3 "" H 1425 4825 50  0001 C CNN
 	1    1425 4825
@@
 F 0 "SW2" V 1475 4725 39  0000 L CNN
 F 1 "DFU" V 1400 4725 39  0000 L CNN
-F 2 "" H 1400 4600 50  0000 C CNN
+F 2 "_div:SMD_Pushbutton_B3U-3100P" H 1400 4600 50  0001 C CNN
 F 3 "" H 1400 4600 50  0000 C CNN
 	1    1400 4600
@@
 Text Notes 875  5300 0    39   ~ 0
 Boot config:\n- Button pushed: DFU bootloader\n- Button released: boot from flash
+NoConn ~ 3525 2925
+Wire Wire Line
+	3950 3225 3525 3225
+Wire Wire Line
+	4200 5475 4750 5475
+NoConn ~ 3525 3425
 $EndSCHEMATC
