File: beacon.kicad_pcb (KiCad board)
At the start: 2 copper layers, 42 x 30 mm, 64 parts, among them SW1 RST, U1 NUF2042XV6, U2 SN65HVD256, U3 MPU-9250, U4 LT1965-3.3, U5 STM32F405RGT6, U6 DWM1000, X1 16MHz

Commit message: Update netlist/layout
Parts:
- added R11: 10k, _std:R_0603, F.Cu at (152.4, 69.6)
- added R12: 10k, _std:R_0603, F.Cu at (125.6, 81.3)
- added SW2: DFU, _div:SMD_Pushbutton_B3U-3100P, F.Cu at (155.5, 67.6)
- moved C9 0.35 mm to (135.8, 81.0)
Connections:
- U5 pad 25: Net-(U5-Pad25) -> /ERROR_LED
- U5 pad 26: /ERROR_LED -> /DEBUG_LED
- U5 pad 27: /DEBUG_LED -> /STATUS_LED
- U5 pad 28: /STATUS_LED -> /BOOT1
- U5 pad 40: Net-(U5-Pad40) -> /UWB_RST_N
- U5 pad 43: /UWB_RST_N -> Net-(U5-Pad43)
- U5 pad 60: GND -> /BOOT0
Routing:
- net /BOOT0: track 0.00 -> 18.6 mm, vias 0 -> 2
- net /BOOT1: track 0.00 -> 8.14 mm
- net VCC: track 166.5 -> 174.5 mm, vias 1 -> 2
- net GND: track 142.4 -> 146.3 mm, vias 15 -> 21
- net /UWB_IRQ: track 39.2 -> 37.5 mm
- net Net-(C9-Pad1): track 7.22 -> 8.18 mm
- net /UWB_RST_N: track 31.2 -> 30.5 mm
Other:
- board text added: "UWB Beacon board v1.1 Club Vaudois de Robotique Autonome cvra.ch"
- board text removed: "UWB Beacon board v1.0 Club Vaudois de Robotique Autonome cvra.ch"
